Commit message: Add odom, map frames and transformations

File: coroco_description/urdf/coroco.xacro (robot description, xacro)
@@ -15,4 +15,11 @@
     <xacro:property name="wheel_length" value="0.1150" />
     <xacro:property name="wheel_radius" value="0.1750" />
+    <!-- static transform between /odom and /base_link -->
+    <link name="odom"/>
+    <joint name="odom_to_base_link=" type="fixed">
+        <origin xyz="0 0 ${-wheel_vertical_offset + wheel_radius}" rpy="0 0 0" />
+        <parent link="odom"/>
+        <child link="base_link"/>
+    </joint>
     <!-- Base link -->
     <link name="base_link">
@@ -27,10 +34,4 @@
             <geometry>
                 <box size="${base_x_size} ${base_y_size} ${base_z_size}"/>
-            </geometry>
-        </collision>
-        <collision>
-            <origin xyz="0 0 ${base_z_size/6}" rpy="0 0 0" />
-            <geometry>
-                <box size="${base_x_size/6} ${base_y_size*1.65} ${base_z_size/3}"/>
             </geometry>
         </collision>

Commit message: Fix model origin point problem

File: coroco_description/urdf/coroco.xacro (robot description, xacro)
@@ -10,7 +10,7 @@
     <xacro:property name="base_y_size" value="0.4400" />
     <xacro:property name="base_z_size" value="0.3100" />
-    <xacro:property name="wheelbase" value="0.5000" />
+    <xacro:property name="wheelbase" value="0.4960" />
     <xacro:property name="track" value="0.4600" />
-    <xacro:property name="wheel_vertical_offset" value="-0.1700" />
+    <xacro:property name="wheel_vertical_offset" value="-0.1575" />
     <xacro:property name="wheel_length" value="0.1150" />
     <xacro:property name="wheel_radius" value="0.1750" />
